File: CH32V003-USB-DevBoard.kicad_sch (KiCad schematic)
At the start: 25 parts, among them J1 USB_C_Receptacle_USB2.0, J2 Conn_01x10, J3 Conn_01x10, J4 Conn_01x01, SW1 SW_Push, U1 ME6211A33M3G-N, U3 CH32V003F4U6, Y1 24MHz

Commit message: Simplify design & switch to TSSOP-20 package for easier assembly
Parts:
- removed JP1, JP2: SolderJumper_2_Open, Library:SolderJumper_0402, symbol Jumper:SolderJumper_2_Open
- R8, R9: value 120R -> 120
- U3: footprint Package_DFN_QFN:QFN-20-1EP_3x3mm_P0.4mm_EP1.65x1.65mm -> Package_SO:ETSSOP-20-1EP_4.4x6.5mm_P0.65mm_EP3x4.2mm
Connections:
- net PA1_H is gone; now on net PA1: J2.5 (Pin_5)
- net PA2_H is gone; now on net PA2: J2.6 (Pin_6)
- net D-: now reaches J1.A7 (D-), J1.B7 (D-), R4.1
- net D+: now reaches J1.A6 (D+), J1.B6 (D+), R5.1
Other:
- moved on the sheet: R4, R5
